Commit message: [feat] update urdf

File: xarm_description/urdf/camera/realsense.gazebo.xacro (robot description, xacro)
@@ -123,3 +123,247 @@
     </gazebo>
   </xacro:macro>
+  <xacro:macro name="realsense_ignition" params="prefix:=''">
+    <gazebo reference="${prefix}camera_depth_frame">
+      <sensor name="${prefix}cameradepth" type="rgbd_camera">
+        <camera name="${prefix}camera">
+          <horizontal_fov>1.57</horizontal_fov>
+          <image>
+            <width>1280</width>
+            <height>720</height>
+            <format>L8</format>
+          </image>
+          <clip>
+            <near>0.1</near>
+            <far>100</far>
+          </clip>
+          <depth_camera>
+            <clip>
+              <near>0.1</near>
+              <far>10</far>
+            </clip>
+          </depth_camera>
+          <noise>
+            <type>gaussian</type>
+            <mean>0.0</mean>
+            <stddev>0.100</stddev>
+          </noise>
+           <!-- <camera_info_topic>${prefix}camera/depth/camera_info</camera_info_topic> -->
+        </camera>
+        <always_on>1</always_on>
+        <update_rate>30</update_rate>
+        <visualize>0</visualize>
+        <topic>${prefix}camera/depth</topic>
+      </sensor>
+    </gazebo>
+    <gazebo reference="${prefix}camera_color_frame">
+      <sensor name="${prefix}cameracolor" type="camera">
+        <!-- <ignition_frame_id>${prefix}camera_color_frame</ignition_frame_id>
+        <optical_frame_id>${prefix}camera_color_frame</optical_frame_id> -->
+        <camera name="${prefix}camera">
+          <horizontal_fov>1.57</horizontal_fov>
+          <image>
+            <width>1280</width>
+            <height>720</height>
+            <format>RGB_INT8</format>
+          </image>
+          <clip>
+            <near>0.1</near>
+            <far>100</far>
+          </clip>
+          <noise>
+            <type>gaussian</type>
+            <mean>0.0</mean>
+            <stddev>0.007</stddev>
+          </noise>
+          <camera_info_topic>${prefix}camera/color/camera_info</camera_info_topic>
+        </camera>
+        <always_on>1</always_on>
+        <update_rate>30</update_rate>
+        <visualize>1</visualize>
+        <topic>${prefix}camera/color/image_raw</topic>
+        <enable_metrics>true</enable_metrics>
+      </sensor>
+    </gazebo>
+    <gazebo reference="${prefix}camera_left_ir_frame">
+      <sensor name="${prefix}cameraired1" type="camera">
+        <camera name="${prefix}camera">
+          <horizontal_fov>1.57</horizontal_fov>
+          <image>
+            <width>1280</width>
+            <height>720</height>
+            <format>L_INT8</format>
+          </image>
+          <clip>
+            <near>0.1</near>
+            <far>100</far>
+          </clip>
+          <noise>
+            <type>gaussian</type>
+            <mean>0.0</mean>
+            <stddev>0.05</stddev>
+          </noise>
+           <camera_info_topic>${prefix}camera/infra1/camera_info</camera_info_topic>
+        </camera>
+        <always_on>1</always_on>
+        <update_rate>30</update_rate>
+        <visualize>0</visualize>
+        <topic>${prefix}camera/infra1/image_raw</topic>
+      </sensor>
+    </gazebo>
+    <gazebo reference="${prefix}camera_right_ir_frame">
+      <sensor name="${prefix}cameraired2" type="camera">
+        <camera name="${prefix}camera">
+          <horizontal_fov>1.57</horizontal_fov>
+          <image>
+            <width>1280</width>
+            <height>720</height>
+            <format>L_INT8</format>
+          </image>
+          <clip>
+            <near>0.1</near>
+            <far>100</far>
+          </clip>
+          <noise>
+            <type>gaussian</type>
+            <mean>0.0</mean>
+            <stddev>0.05</stddev>
+          </noise>
+          <camera_info_topic>${prefix}camera/infra2/camera_info</camera_info_topic>
+        </camera>
+        <always_on>1</always_on>
+        <update_rate>30</update_rate>
+        <visualize>0</visualize>
+        <topic>${prefix}camera/infra2/image_raw</topic>
+      </sensor>
+    </gazebo>
+    <gazebo>
+      <plugin
+        filename="libignition-gazebo-sensors-system.so"
+        name="ignition::gazebo::systems::Sensors">
+        <render_engine>ogre2</render_engine>
+      </plugin>
+    </gazebo>
+  </xacro:macro>
+  <xacro:macro name="realsense_gz" params="prefix:=''">
+    <gazebo reference="${prefix}camera_depth_frame">
+      <sensor name="${prefix}cameradepth" type="rgbd_camera">
+        <camera name="${prefix}camera">
+          <horizontal_fov>1.57</horizontal_fov>
+          <image>
+            <width>1280</width>
+            <height>720</height>
+            <format>L8</format>
+          </image>
+          <clip>
+            <near>0.1</near>
+            <far>100</far>
+          </clip>
+          <depth_camera>
+            <clip>
+              <near>0.1</near>
+              <far>10</far>
+            </clip>
+          </depth_camera>
+          <noise>
+            <type>gaussian</type>
+            <mean>0.0</mean>
+            <stddev>0.100</stddev>
+          </noise>
+           <!-- <camera_info_topic>${prefix}camera/depth/camera_info</camera_info_topic> -->
+        </camera>
+        <always_on>1</always_on>
+        <update_rate>30</update_rate>
+        <visualize>0</visualize>
+        <topic>${prefix}camera/depth</topic>
+      </sensor>
+    </gazebo>
+    <gazebo reference="${prefix}camera_color_frame">
+      <sensor name="${prefix}cameracolor" type="camera">
+        <!-- <ignition_frame_id>${prefix}camera_color_frame</ignition_frame_id>
+        <optical_frame_id>${prefix}camera_color_frame</optical_frame_id> -->
+        <camera name="${prefix}camera">
+          <horizontal_fov>1.57</horizontal_fov>
+          <image>
+            <width>1280</width>
+            <height>720</height>
+            <format>RGB_INT8</format>
+          </image>
+          <clip>
+            <near>0.1</near>
+            <far>100</far>
+          </clip>
+          <noise>
+            <type>gaussian</type>
+            <mean>0.0</mean>
+            <stddev>0.007</stddev>
+          </noise>
+          <camera_info_topic>${prefix}camera/color/camera_info</camera_info_topic>
+        </camera>
+        <always_on>1</always_on>
+        <update_rate>30</update_rate>
+        <visualize>1</visualize>
+        <topic>${prefix}camera/color/image_raw</topic>
+        <enable_metrics>true</enable_metrics>
+      </sensor>
+    </gazebo>
+    <gazebo reference="${prefix}camera_left_ir_frame">
+      <sensor name="${prefix}cameraired1" type="camera">
+        <camera name="${prefix}camera">
+          <horizontal_fov>1.57</horizontal_fov>
+          <image>
+            <width>1280</width>
+            <height>720</height>
+            <format>L_INT8</format>
+          </image>
+          <clip>
+            <near>0.1</near>
+            <far>100</far>
+          </clip>
+          <noise>
+            <type>gaussian</type>
+            <mean>0.0</mean>
+            <stddev>0.05</stddev>
+          </noise>
+           <camera_info_topic>${prefix}camera/infra1/camera_info</camera_info_topic>
+        </camera>
+        <always_on>1</always_on>
+        <update_rate>30</update_rate>
+        <visualize>0</visualize>
+        <topic>${prefix}camera/infra1/image_raw</topic>
+      </sensor>
+    </gazebo>
+    <gazebo reference="${prefix}camera_right_ir_frame">
+      <sensor name="${prefix}cameraired2" type="camera">
+        <camera name="${prefix}camera">
+          <horizontal_fov>1.57</horizontal_fov>
+          <image>
+            <width>1280</width>
+            <height>720</height>
+            <format>L_INT8</format>
+          </image>
+          <clip>
+            <near>0.1</near>
+            <far>100</far>
+          </clip>
+          <noise>
+            <type>gaussian</type>
+            <mean>0.0</mean>
+            <stddev>0.05</stddev>
+          </noise>
+          <camera_info_topic>${prefix}camera/infra2/camera_info</camera_info_topic>
+        </camera>
+        <always_on>1</always_on>
+        <update_rate>30</update_rate>
+        <visualize>0</visualize>
+        <topic>${prefix}camera/infra2/image_raw</topic>
+      </sensor>
+    </gazebo>
+    <gazebo>
+      <plugin
+        filename="libgz-sim-sensors-system.so"
+        name="gz::sim::systems::Sensors">
+        <render_engine>ogre2</render_engine>
+      </plugin>
+    </gazebo>
+  </xacro:macro>
 </robot>

File: xarm_description/urdf/common/common.gazebo.xacro (robot description, xacro)
@@ -1,4 +1,13 @@
 <?xml version="1.0"?>
 <robot xmlns:xacro="http://ros.org/wiki/xacro">
+  <xacro:macro name="gz_ros2_control_plugin" params="ros2_control_params:=''">
+    <gazebo>
+      <plugin filename="gz_ros2_control-system" name="gz_ros2_control::GazeboSimROS2ControlPlugin">
+        <xacro:if value="${ros2_control_params != ''}">
+          <parameters>${ros2_control_params}</parameters>
+        </xacro:if>
+      </plugin>
+    </gazebo>
+  </xacro:macro>
   <xacro:macro name="ignition_ros2_control_plugin" params="prefix:='' ros2_control_params:=''">
     <gazebo>

File: xarm_description/urdf/gripper/xarm_gripper.gazebo.xacro (robot description, xacro)
@@ -2,5 +2,5 @@
 <robot xmlns:xacro="http://ros.org/wiki/xacro">
   <!-- from mimic_joint_gazebo_tutorial by @mintar, refer: https://github.com/mintar/mimic_joint_gazebo_tutorial -->
-  <xacro:macro name="mimic_joint_plugin_gazebo" params="name_prefix following_joint mimic_joint has_pid:=false multiplier:=1.0 offset:=0 sensitiveness:=0.0 max_effort:=1.0 robot_namespace:=''">
+  <xacro:macro name="mimic_joint_plugin_gazebo" params="name_prefix following_joint mimic_joint has_pid:=false multiplier:=1.0 offset:=0 sensitiveness:=0.0 max_effort:=1.0 ros2_control_plugin:='gazebo_ros2_control/GazeboSystem' robot_namespace:=''">
     <!-- ros2 -->
     <xacro:if value="${is_ros2}">
@@ -12,6 +12,12 @@
       <!-- <xacro:property name="filename" value="libroboticsgroup_upatras_gazebo_mimic_joint_plugin.so" /> -->
     </xacro:unless>
+    <xacro:if value="${ros2_control_plugin == 'gazebo_ros2_control/GazeboSystem'}">
+      <xacro:property name="plugin_name" value="${name_prefix}mimic_joint_plugin" />
+    </xacro:if>
+    <xacro:unless value="${ros2_control_plugin == 'gazebo_ros2_control/GazeboSystem'}">
+      <xacro:property name="plugin_name" value="gz::sim::systems::GazeboMimicJointPlugin" />
+    </xacro:unless>
     <gazebo>
-      <plugin name="${name_prefix}mimic_joint_plugin" filename="${filename}">
+      <plugin name="${plugin_name}" filename="${filename}">
         <joint>${following_joint}</joint>
         <mimicJoint>${mimic_joint}</mimicJoint>

File: xarm_description/urdf/gripper/xarm_gripper_macro.xacro (robot description, xacro)
@@ -20,17 +20,17 @@
     <xacro:mimic_joint_plugin_gazebo name_prefix="${prefix}left_finger_joint"
       following_joint="${prefix}drive_joint" mimic_joint="${prefix}left_finger_joint"
-      has_pid="${is_ros2}" multiplier="1.0" max_effort="10.0" />
+      has_pid="${is_ros2}" multiplier="1.0" max_effort="10.0" ros2_control_plugin="${ros2_control_plugin}"/>
     <xacro:mimic_joint_plugin_gazebo name_prefix="${prefix}left_inner_knuckle_joint"
       following_joint="${prefix}drive_joint" mimic_joint="${prefix}left_inner_knuckle_joint"
-      has_pid="${is_ros2}" multiplier="1.0" max_effort="10.0" />
+      has_pid="${is_ros2}" multiplier="1.0" max_effort="10.0" ros2_control_plugin="${ros2_control_plugin}"/>
     <xacro:mimic_joint_plugin_gazebo name_prefix="${prefix}right_outer_knuckle_joint"
       following_joint="${prefix}drive_joint" mimic_joint="${prefix}right_outer_knuckle_joint"
-      has_pid="${is_ros2}" multiplier="1.0" max_effort="10.0" />
+      has_pid="${is_ros2}" multiplier="1.0" max_effort="10.0" ros2_control_plugin="${ros2_control_plugin}"/>
     <xacro:mimic_joint_plugin_gazebo name_prefix="${prefix}right_finger_joint"
       following_joint="${prefix}drive_joint" mimic_joint="${prefix}right_finger_joint"
-      has_pid="${is_ros2}" multiplier="1.0" max_effort="10.0" />
+      has_pid="${is_ros2}" multiplier="1.0" max_effort="10.0" ros2_control_plugin="${ros2_control_plugin}"/>
     <xacro:mimic_joint_plugin_gazebo name_prefix="${prefix}right_inner_knuckle_joint"
       following_joint="${prefix}drive_joint" mimic_joint="${prefix}right_inner_knuckle_joint"
-      has_pid="${is_ros2}" multiplier="1.0" max_effort="10.0" />
+      has_pid="${is_ros2}" multiplier="1.0" max_effort="10.0" ros2_control_plugin="${ros2_control_plugin}"/>
   </xacro:macro>
 </robot>

File: xarm_description/urdf/xarm_device_macro.xacro (robot description, xacro)
@@ -52,9 +52,9 @@
     <!-- Specify Mesh file path -->
     <xacro:property name="mesh_suffix" value="${mesh_suffix}" scope="parent"/>
-    <xacro:if value="${ros2_control_plugin == 'gazebo_ros2_control/GazeboSystem' or ros2_control_plugin == 'ign_ros2_control/IgnitionSystem'}">
+    <xacro:if value="${ros2_control_plugin == 'gazebo_ros2_control/GazeboSystem' or ros2_control_plugin == 'ign_ros2_control/IgnitionSystem' or ros2_control_plugin == 'gz_ros2_control/GazeboSimSystem'}">
       <!-- gazebo use -->
       <xacro:property name="mesh_path" value="file://$(find xarm_description)/meshes" scope="parent"/>
     </xacro:if>
-    <xacro:unless value="${ros2_control_plugin == 'gazebo_ros2_control/GazeboSystem' or ros2_control_plugin == 'ign_ros2_control/IgnitionSystem'}">
+    <xacro:unless value="${ros2_control_plugin == 'gazebo_ros2_control/GazeboSystem' or ros2_control_plugin == 'ign_ros2_control/IgnitionSystem' or ros2_control_plugin == 'gz_ros2_control/GazeboSimSystem'}">
       <xacro:property name="mesh_path" value="package://xarm_description/meshes" scope="parent"/>
     </xacro:unless>
@@ -207,5 +207,13 @@
       <xacro:if value="${add_d435i_links}">
         <xacro:include filename="$(find xarm_description)/urdf/camera/realsense.gazebo.xacro" />
-        <xacro:realsense_gazebo prefix="${prefix}" />
+        <xacro:if value="${ros2_control_plugin == 'gz_ros2_control/GazeboSimSystem'}">
+          <xacro:realsense_gz prefix="${prefix}" />
+        </xacro:if>
+        <xacro:if value="${ros2_control_plugin == 'ign_ros2_control/IgnitionSystem'}">
+          <xacro:realsense_ignition prefix="${prefix}" />
+        </xacro:if>
+        <xacro:if value="${ros2_control_plugin == 'gazebo_ros2_control/GazeboSystem'}">
+          <xacro:realsense_gazebo prefix="${prefix}" />
+        </xacro:if>
       </xacro:if>
     </xacro:if>
